File: PCB Files/Ocean Harness.kicad_pcb (KiCad board)
At the start: 4 copper layers, 115.8 x 75.2 mm, 24 parts, among them J1 JAE DX07S024XJ1R1100, J3 Molex 0346910200, J4 Molex 0346910200, J5 Molex 0346910162, J6 Molex 0346910162, K1 G5V-2-H1 DC12, U1 Vishay DG419LEDY-T1-GE4, U2 Vishay DG419LEDY-T1-GE4

Commit message: Add R5 dropper to schematic and link its footprint on the board
R5 (160R 0805) replaces the U3 L78L12 as the relay coil / switch supply
dropper. The symbol was added to the schematic and the footprint had been
hand-placed in the PCB editor, but the footprint carried no (path ...) link
to the schematic symbol, so "Update PCB from Schematic" could not match the
two and wanted to add a second R5.

Linking the existing footprint (rather than letting the update drop in a new
one) keeps its placement and its /12V_PROT and VIN traces. KiCad then filled
in the footprint library id, description, pad pintypes and unit metadata on
the next update, and refilled the copper zones.

Also carried over from the working copy: relay datasheet corrected to
G5V-2-H1 DC12, an "<---- ADAS ECU" silkscreen marker, and reference-
designator text repositioning.

Co-Authored-By: Claude Opus 5 <noreply@anthropic.com>
Parts:
- R5: footprint R_0805_2012Metric -> Resistor_SMD:R_0805_2012Metric
Connections:
- J1 pad S2: GND -> (no net)
- J1 pad S3: GND -> (no net)
- J1 pad S4: GND -> (no net)
Other:
- board text added: "<---- ADAS ECU"
Changed lines of the file:
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@@
 		(tags "346910200 ")
 		(property "Reference" "J3"
-			(at 11.43 1.27 90)
+			(at 11.315394 -3.548602 90)
 			(unlocked yes)
 			(layer "F.SilkS")
@@
 		(tags "346910162 ")
 		(property "Reference" "J6"
-			(at 8.89 1.27 270)
+			(at 8.89 -3.965434 270)
 			(unlocked yes)
 			(layer "F.SilkS")
@@
 			(layers "*.Cu" "*.Mask")
 			(remove_unused_layers no)
-			(net "GND")
 			(solder_mask_margin 0.102)
 		)
@@
 			(layers "*.Cu" "*.Mask")
 			(remove_unused_layers no)
-			(net "GND")
 			(solder_mask_margin 0.102)
 		)
@@
 			(layers "*.Cu" "*.Mask")
 			(remove_unused_layers no)
-			(net "GND")
 			(solder_mask_margin 0.102)
 		)
@@
 		(tags "346910162 ")
 		(property "Reference" "J5"
-			(at 8.89 1.27 90)
+			(at 8.775394 -4.048602 90)
 			(unlocked yes)
 			(layer "F.SilkS")
@@
 			)
 		)
-		(property "Datasheet" "G5V-2 DC12"
+		(property "Datasheet" "G5V-2-H1 DC12"
 			(at 0 0 0)
 			(layer "F.Fab")
@@
 		)
 	)
-	(footprint "R_0805_2012Metric"
+	(footprint "Resistor_SMD:R_0805_2012Metric"
 		(layer "F.Cu")
 		(at 126.066 73.406 90)
@@
 			)
 		)
-		(property "Description" ""
+		(property "Description" "Relay coil / switch supply dropper, replaces U3 L78L12"
 			(at 0 0 90)
 			(layer "F.Fab")
@@
 			)
 		)
+		(property ki_fp_filters "R_*")
+		(sheetname "/")
+		(sheetfile "Ocean Harness.kicad_sch")
+		(units
+			(unit
+				(name "A")
+				(pins "1" "2")
+			)
+		)
 		(attr smd)
 		(duplicate_pad_numbers_are_jumpers no)
@@
 			(roundrect_rratio 0.243902)
 			(net "/12V_PROT")
+			(pintype "passive")
 		)
 		(pad "2" smd roundrect
@@
 			(roundrect_rratio 0.243902)
 			(net "VIN")
+			(pintype "passive")
 		)
 		(embedded_fonts no)
@@
 		(tags "346910200 ")
 		(property "Reference" "J4"
-			(at 11.43 1.27 270)
+			(at 11.566321 -3.465434 270)
 			(unlocked yes)
 			(layer "F.SilkS")
@@
 		(layer "Edge.Cuts")
 	)
+	(gr_text "<---- ADAS ECU"
+		(at 84.5 74.5 0)
+		(layer "F.SilkS")
+		(effects
+			(font
+				(size 1.5 1.5)
+				(thickness 0.3)
+				(bold yes)
+			)
+			(justify left bottom)
+		)
+	)
 	(segment
 		(start 114.534566 82.683679)
@@
 		(start 164.674606 104.565394)
 		(end 166.048602 104.565394)
-		(width 2.4)
+		(width 1)
 		(layer "B.Cu")
 		(net "/Harness_12v")
@@
 		(start 176.022 74.422)
 		(end 176.022 104.648)
-		(width 4)
+		(width 1)
 		(layer "B.Cu")
 		(net "/Harness_12v")
@@
 		(start 173.736 72.136)
 		(end 176.022 74.422)
-		(width 4)
+		(width 1)
 		(layer "B.Cu")
 		(net "/Harness_12v")
@@
 		(start 114.534566 82.683679)
 		(end 125.082245 72.136)
-		(width 2.1)
+		(width 1)
 		(layer "B.Cu")
 		(net "/Harness_12v")
@@
 		(start 176.022 104.648)
 		(end 170.18 110.49)
-		(width 3)
+		(width 1)
 		(layer "B.Cu")
 		(net "/Harness_12v")
@@
 		(start 125.082245 72.136)
 		(end 173.736 72.136)
-		(width 1.95)
+		(width 1)
 		(layer "B.Cu")
 		(net "/Harness_12v")
@@
 		(start 170.18 110.49)
 		(end 164.592 110.49)
-		(width 3)
+		(width 1)
 		(layer "B.Cu")
 		(net "/Harness_12v")
@@
 		(start 163.068 106.172)
 		(end 164.674606 104.565394)
-		(width 3.4)
+		(width 1)
 		(layer "B.Cu")
 		(net "/Harness_12v")
@@
 		(start 164.592 110.49)
 		(end 163.068 108.966)
-		(width 2.9)
+		(width 1)
 		(layer "B.Cu")
 		(net "/Harness_12v")
@@
 		(start 163.068 108.966)
 		(end 163.068 106.172)
-		(width 2.5)
+		(width 1)
 		(layer "B.Cu")
 		(net "/Harness_12v")
