File: PCB Files/Ocean Harness.kicad_pcb (KiCad board)
At the start: 4 copper layers, 115.8 x 75.2 mm, 24 parts, among them J1 JAE DX07S024XJ1R1100, J3 Molex 0346910200, J4 Molex 0346910200, J5 Molex 0346910162, J6 Molex 0346910162, K1 G5V-2-H1 DC12, U1 Vishay DG419LEDY-T1-GE4, U2 Vishay DG419LEDY-T1-GE4

Commit message: Fix production blockers: zone fills, fiducials, MPNs, polarity marks, via rings
Addresses the five pre-fab blockers from design_review_2026-10-13.md. No
track, pad, footprint position or net was modified -- net membership is
identical across all 70 nets, all 24 original footprints have unchanged
pad-to-net maps, and ERC is unchanged at 76 warnings / 0 errors.

- Refill zones. As committed previously the board had stale fills, leaving
  all four J1 USB-C shield pads unconnected to the GND pour; gerbers plotted
  from it would have shipped an ungrounded shield. DRC now reports 0
  unconnected items without needing --refill-zones.

- Add fiducials FID1-FID3 on F.Cu (standard Fiducial_1mm_Mask2mm, 1 mm
  copper / 2 mm mask opening). Placed as a scalene non-symmetric triangle in
  the open middle band -- the J3-J6 housings cover the outer thirds of the
  top surface, so corner fiducials would sit under a connector body. Clears
  FD-001.

- Populate MPN / Manufacturer / Spec fields on 22 symbols and mirror them
  onto the PCB footprints. Coverage 0/13 -> 10/13; SS-001 (blocker) is now
  SS-002 (warning). D10 is specified as the onsemi SS34 because the
  footprint is SMA (DO-214AC) and Vishay's SS34 is SMC and will not fit.
  The Molex connectors carry an explicit note to verify the polarization
  code against the Fisker CON1 keying. C1, C2 and R5 are jellybean parts
  left for a house part number; their full spec is recorded in Spec.

- Add cathode polarity markers to D9/D11 on F.SilkS and F.Fab. The
  My_Components:SMAJ16A footprint drew only a plain rectangle, so a
  reversed TVS -- which dead-shorts the 12 V rail -- had no board-level
  reference. D9's bar sits below the body because its left side carries the
  incoming 12V_PROT feed; D11's sits to the left. Both carry an identical
  fab-layer bar. The library footprint itself is still defective.

- Grow 25 of 27 vias from 0.5 to 0.6 mm so the annular ring reaches 0.15 mm
  and meets IPC-6012 Class 2. The vias at (145.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
Parts:
- added FID1: Fiducial_1mm_Mask2mm, Fiducial:Fiducial_1mm_Mask2mm, F.Cu at (121.2, 89.2)
- added FID2: Fiducial_1mm_Mask2mm, Fiducial:Fiducial_1mm_Mask2mm, F.Cu at (129.8, 44.8)
- added FID3: Fiducial_1mm_Mask2mm, Fiducial:Fiducial_1mm_Mask2mm, F.Cu at (160.8, 97.8)
