File: PCB Files/Ocean Harness.kicad_sch (KiCad schematic)
At the start: 22 parts, among them J1 JAE DX07S024XJ1R1100, J3 Molex 0346910200, J4 Molex 0346910200, J5 Molex 0346910162, J6 Molex 0346910162, K1 G5V-2 DC12, U1 Vishay DG419LEDY-T1-GE4, U2 Vishay DG419LEDY-T1-GE4, U3 L78L12_SOT89

Commit message: Restructure to match passthrough-harness-box repo format; update board
Bring the repo in line with the volvo-polestar-passthrough-harness-box
layout: a 3D models/ directory with a render and STEP export, an
analysis/ manifest under PCB Files/, a dated design review, and a README
that describes the board rather than stubbing it.

Board changes made during the review, all with DRC and ERC at 0 errors:

- K1 changed to Omron G5V-2-H1 DC12 (960 R / 12.5 mA / 150 mW coil,
  180% max coil voltage). Package-identical to the G5V-2, so the
  footprint and 3D model carry over unchanged.
- U3 (L78L12) removed, replaced by R5 in the same footprint position.
  The part could never regulate: it needs >=14.5 V in and the DC-DC
  gives 13.4-14.1 V after the SS34 drop. R5 is 160 R, sized for the
  H1's 960 R coil.
- VBAT pass-through widened per segment, 61.4 mOhm -> 24.6 mOhm.
- Two M3 mounting holes added; the board previously had none.
- Redundant J1 Edge.Cuts cutout deleted, clearing 3 copper_edge_clearance
  errors. The library footprint still has the defect.
- 3D models added to J3/J4/J5/J6, sourced from Ocean Conversion PCB.

Co-Authored-By: Claude Opus 5 <noreply@anthropic.com>
Parts:
- removed U3: L78L12_SOT89, Package_TO_SOT_SMD:SOT-89-3, symbol Regulator_Linear:L78L12_SOT89
- added R5: 160, Resistor_SMD:R_0805_2012Metric, symbol Device:R
- D9: value 16V -> SMAJ16A
- K1: value G5V-2 DC12 -> G5V-2-H1 DC12
Connections:
- net 12V_PROT: now also R5.1
- net VIN: now also R5.2
Changed lines of the file:
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@@
 	(wire
 		(pts
-			(xy 309.88 164.084) (xy 299.72 164.084)
+			(xy 313.69 164.084) (xy 299.72 164.084)
 		)
 		(stroke
@@
 	(wire
 		(pts
-			(xy 325.12 164.084) (xy 327.66 164.084)
+			(xy 321.31 164.084) (xy 327.66 164.084)
 		)
 		(stroke
@@
 	(wire
 		(pts
-			(xy 317.5 171.704) (xy 317.5 174.244)
-		)
-		(stroke
-			(width 0)
-			(type default)
-		)
-	)
-	(wire
-		(pts
 			(xy 130.81 95.25) (xy 139.7 95.25)
 		)
@@
 		)
 	)
-	(label "GND"
-		(at 317.5 174.244 0)
-		(effects
-			(font
-				(size 1.27 1.27)
-			)
-			(justify left bottom)
-		)
-	)
 	(label "SBU 1"
 		(at 97.79 30.48 180)
@@
 			)
 		)
-		(property "Value" "16V"
+		(property "Value" "SMAJ16A"
 			(at 193.799 168.656 90)
 			(show_name no)
@@
 	)
 	(symbol
-		(lib_id "power:GND")
+		(lib_id "power:VCC")
 		(at 139.7 90.17 0)
-		(mirror x)
 		(unit 1)
 		(body_style 1)
@@
 			)
 		)
-		(property "Description" "Power symbol creates a global label with name \"GND\" , ground"
+		(property "Description" "Power symbol creates a global label with name \"VCC\""
 			(at 139.7 90.17 0)
 			(hide yes)
@@
 		)
 	)
+	(wire
+		(pts
+			(xy 327.66 164.084) (xy 327.66 158.75)
+		)
+		(stroke
+			(width 0)
+			(type default)
+		)
+	)
 	(symbol
-		(lib_id "Regulator_Linear:L78L12_SOT89")
-		(at 317.5 164.084 0)
+		(lib_id "power:PWR_FLAG")
+		(at 327.66 158.75 0)
 		(unit 1)
 		(body_style 1)
@@
 		(in_pos_files yes)
 		(dnp no)
-		(property "Reference" "U3"
-			(at 317.5 159.004 0)
+		(property "Reference" "#FLG03"
+			(at 327.66 156.845 0)
+			(hide yes)
 			(show_name no)
 			(do_not_autoplace no)
@@
 			)
 		)
-		(property "Value" "L78L12_SOT89"
-			(at 308.102 172.212 0)
+		(property "Value" "PWR_FLAG"
+			(at 327.406 154.432 0)
 			(show_name no)
 			(do_not_autoplace no)
@@
 			)
 		)
-		(property "Footprint" "Package_TO_SOT_SMD:SOT-89-3"
-			(at 317.5 164.084 0)
+		(property "Footprint" ""
+			(at 327.66 158.75 0)
+			(hide yes)
+			(show_name no)
+			(do_not_autoplace no)
+			(effects
+				(font
+					(size 1.27 1.27)
+				)
+			)
+		)
+		(property "Datasheet" ""
+			(at 327.66 158.75 0)
+			(hide yes)
+			(show_name no)
+			(do_not_autoplace no)
+			(effects
+				(font
+					(size 1.27 1.27)
+				)
+			)
+		)
+		(property "Description" "Special symbol for telling ERC where power comes from"
+			(at 327.66 158.75 0)
+			(hide yes)
+			(show_name no)
+			(do_not_autoplace no)
+			(effects
+				(font
+					(size 1.27 1.27)
+				)
+			)
+		)
+		(pin "1"
+		)
+		(instances
+			(project "Ocean Harness"
+				(path "/9bff95d7-5e0b-4644-a7b2-cd392dfbdb8f"
+					(reference "#FLG03")
+					(unit 1)
+				)
+			)
+		)
+	)
+	(symbol
+		(lib_id "Device:R")
+		(at 317.5 164.084 90)
+		(unit 1)
+		(body_style 1)
+		(exclude_from_sim no)
+		(in_bom yes)
+		(on_board yes)
+		(in_pos_files yes)
+		(dnp no)
+		(property "Reference" "R5"
+			(at 317.5 160.274 0)
+			(show_name no)
+			(do_not_autoplace no)
+			(effects
+				(font
+					(size 1.27 1.27)
+				)
+			)
+		)
+		(property "Value" "160"
+			(at 317.5 167.894 0)
+			(show_name no)
+			(do_not_autoplace no)
+			(effects
+				(font
+					(size 1.27 1.27)
+				)
+			)
+		)
+		(property "Footprint" "Resistor_SMD:R_0805_2012Metric"
+			(at 317.5 164.084 90)
 			(hide yes)
 			(show_name no)
@@
 		(property "Datasheet" ""
 			(at 317.5 164.084 0)
+			(hide yes)
 			(show_name no)
 			(do_not_autoplace no)
@@
 			)
 		)
-		(property "Description" ""
+		(property "Description" "Relay coil / switch supply dropper, replaces U3 L78L12"
 			(at 317.5 164.084 0)
+			(hide yes)
 			(show_name no)
 			(do_not_autoplace no)
@@
 		(pin "2"
 		)
-		(pin "3"
-		)
 		(instances
 			(project "Ocean Harness"
 				(path "/9bff95d7-5e0b-4644-a7b2-cd392dfbdb8f"
-					(reference "U3")
+					(reference "R5")
 					(unit 1)
 				)
@@
 			)
 		)
-		(property "Value" "G5V-2 DC12"
+		(property "Value" "G5V-2-H1 DC12"
 			(at 109.982 104.648 0)
 			(show_name no)
@@
 			)
 		)
-		(property "Datasheet" "G5V-2 DC12"
+		(property "Datasheet" "G5V-2-H1 DC12"
 			(at 90.17 90.17 0)
 			(hide yes)

Commit message: Fix production blockers: zone fills, fiducials, MPNs, polarity marks, via rings
Addresses the five pre-fab blockers from design_review_2026-10-13.md. No
track, pad, footprint position or net was modified -- net membership is
identical across all 70 nets, all 24 original footprints have unchanged
pad-to-net maps, and ERC is unchanged at 76 warnings / 0 errors.

- Refill zones. As committed previously the board had stale fills, leaving
  all four J1 USB-C shield pads unconnected to the GND pour; gerbers plotted
  from it would have shipped an ungrounded shield. DRC now reports 0
  unconnected items without needing --refill-zones.

- Add fiducials FID1-FID3 on F.Cu (standard Fiducial_1mm_Mask2mm, 1 mm
  copper / 2 mm mask opening). Placed as a scalene non-symmetric triangle in
  the open middle band -- the J3-J6 housings cover the outer thirds of the
  top surface, so corner fiducials would sit under a connector body. Clears
  FD-001.

- Populate MPN / Manufacturer / Spec fields on 22 symbols and mirror them
  onto the PCB footprints. Coverage 0/13 -> 10/13; SS-001 (blocker) is now
  SS-002 (warning). D10 is specified as the onsemi SS34 because the
  footprint is SMA (DO-214AC) and Vishay's SS34 is SMC and will not fit.
  The Molex connectors carry an explicit note to verify the polarization
  code against the Fisker CON1 keying. C1, C2 and R5 are jellybean parts
  left for a house part number; their full spec is recorded in Spec.

- Add cathode polarity markers to D9/D11 on F.SilkS and F.Fab. The
  My_Components:SMAJ16A footprint drew only a plain rectangle, so a
  reversed TVS -- which dead-shorts the 12 V rail -- had no board-level
  reference. D9's bar sits below the body because its left side carries the
  incoming 12V_PROT feed; D11's sits to the left. Both carry an identical
  fab-layer bar. The library footprint itself is still defective.

- Grow 25 of 27 vias from 0.5 to 0.6 mm so the annular ring reaches 0.15 mm
  and meets IPC-6012 Class 2. The vias at (145.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
Parts:
- C1: Spec (none) -> Capacitor, 0.33uF, >=50V, X7R, 0603 -- assign house part be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
- C2: Spec (none) -> Capacitor, 0.1uF, >=50V, X7R, 0603 -- assign house part bef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
- CR1: MPN (none) -> 1N4148W-7-F; Manufacturer (none) -> Diodes Incorporated; Spec (none) -> Diode, switching, 100V 150mA, SOD-123
- D1, D2, D3, D8: MPN (none) -> PESD1CAN,215; Manufacturer (none) -> Nexperia; Spec (none) -> ESD protection diode array for CAN, SOT-23
- D10: MPN (none) -> SS34; Manufacturer (none) -> onsemi; Spec (none) -> Schottky rectifier 40V 3A. MUST be DO-214AC (SMA) -- Vishay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
- D11, D9: MPN (none) -> SMAJ16A; Manufacturer (none) -> Littelfuse; Spec (none) -> TVS diode, unidirectional, 16V standoff, DO-214AC (SMA). Ca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
- J1: MPN (none) -> DX07S024XJ1R1100; Manufacturer (none) -> JAE Electronics; Spec (none) -> USB Type-C receptacle, 24 position, to comma device
- J3: MPN (none) -> 34691-0200; Manufacturer (none) -> Molex; Spec (none) -> Stac64 header, 20 circuit, CON1 section A, harness side. VE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
- J4: MPN (none) -> 34691-0200; Manufacturer (none) -> Molex; Spec (none) -> Stac64 header, 20 circuit, CON1 section A, ECU side. VERIFY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
- J5: MPN (none) -> 34691-0162; Manufacturer (none) -> Molex; Spec (none) -> Stac64 header, 16 circuit, CON1 section B, harness side. VE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
- J6: MPN (none) -> 34691-0162; Manufacturer (none) -> Molex; Spec (none) -> Stac64 header, 16 circuit, CON1 section B, ECU side. VERIFY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
- K1: MPN (none) -> G5V-2-H1 DC12; Manufacturer (none) -> Omron; Spec (none) -> Signal relay, DPDT, 12VDC high-sensitivity coil (960 ohm, 1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
- R2, R3, R4: MPN (none) -> ESR03EZPJ121; Manufacturer (none) -> ROHM; Spec (none) -> Resistor, 120 ohm 5%, anti-surge
- R5: Spec (none) -> Resistor, 160 ohm, 1%, >=0.125W, 0805 -- relay coil dropper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
- U1, U2: MPN (none) -> DG419LEDY-T1-GE4; Manufacturer (none) -> Vishay Siliconix; Spec (none) -> Analog switch, SPDT, single supply, SOIC-8
